File: src/pcb/GCCMX.kicad_sch (KiCad schematic)
At the start: 24 parts, among them J1 Conn_01x04, J2 Conn_01x04, SW1 SW_SPST, SW10 SW_SPST, SW11 SW_SPST, SW12 SW_SPST, SW13 SW_SPST, SW14 SW_SPST, SW15 SW_SPST, SW16 SW_SPST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

Commit message: updates
Parts:
- removed D1: 1N5817, Diode_THT:D_DO-41_SOD81_P10.16mm_Horizontal, symbol Diode:1N5817
Connections:
- net GND: now also U1.13 (GND), U1.18 (GND), U1.23 (GND), U1.28 (GND), U1.3 (GND), U1.8 (GND)
- net at U1.39 (VSYS): now also J2.3 (Pin_3)
Changed lines of the file:
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@@
 (kicad_sch (version 20211123) (generator eeschema)
   (paper "A4")
+  (junction (at 152.4 138.43) (diameter 0) (color 0 0 0 0)
+  )
   (junction (at 198.12 137.16) (diameter 0) (color 0 0 0 0)
   )
+  (junction (at 83.82 138.43) (diameter 0) (color 0 0 0 0)
+  )
+  (junction (at 83.82 151.13) (diameter 0) (color 0 0 0 0)
+  )
   (junction (at 152.4 113.03) (diameter 0) (color 0 0 0 0)
   )
@@
   (junction (at 152.4 125.73) (diameter 0) (color 0 0 0 0)
   )
+  (junction (at 152.4 153.67) (diameter 0) (color 0 0 0 0)
+  )
   (junction (at 198.12 111.76) (diameter 0) (color 0 0 0 0)
   )
@@
   (junction (at 198.12 22.86) (diameter 0) (color 0 0 0 0)
   )
+  (junction (at 83.82 125.73) (diameter 0) (color 0 0 0 0)
+  )
   (junction (at 198.12 60.96) (diameter 0) (color 0 0 0 0)
   )
+  (junction (at 152.4 151.13) (diameter 0) (color 0 0 0 0)
+  )
   (junction (at 198.12 153.67) (diameter 0) (color 0 0 0 0)
   )
-  (wire (pts (xy 135.89 110.49) (xy 139.7 110.49))
+  (wire (pts (xy 151.13 91.44) (xy 157.48 91.44))
     (stroke (width 0) (type default) (color 0 0 0 0))
   )
@@
     (stroke (width 0) (type default) (color 0 0 0 0))
   )
+  (wire (pts (xy 100.33 138.43) (xy 83.82 138.43))
+    (stroke (width 0) (type default) (color 0 0 0 0))
+  )
+  (wire (pts (xy 152.4 151.13) (xy 152.4 153.67))
+    (stroke (width 0) (type default) (color 0 0 0 0))
+  )
   (wire (pts (xy 198.12 48.26) (xy 195.58 48.26))
     (stroke (width 0) (type default) (color 0 0 0 0))
@@
     (stroke (width 0) (type default) (color 0 0 0 0))
   )
+  (wire (pts (xy 83.82 138.43) (xy 83.82 151.13))
+    (stroke (width 0) (type default) (color 0 0 0 0))
+  )
   (wire (pts (xy 219.71 149.86) (xy 210.82 149.86))
     (stroke (width 0) (type default) (color 0 0 0 0))
@@
     (stroke (width 0) (type default) (color 0 0 0 0))
   )
+  (wire (pts (xy 152.4 138.43) (xy 152.4 151.13))
+    (stroke (width 0) (type default) (color 0 0 0 0))
+  )
   (wire (pts (xy 100.33 146.05) (xy 91.44 146.05))
     (stroke (width 0) (type default) (color 0 0 0 0))
   )
-  (wire (pts (xy 149.86 110.49) (xy 149.86 88.9))
-    (stroke (width 0) (type default) (color 0 0 0 0))
-  )
   (wire (pts (xy 198.12 137.16) (xy 200.66 137.16))
     (stroke (width 0) (type default) (color 0 0 0 0))
@@
     (stroke (width 0) (type default) (color 0 0 0 0))
   )
-  (wire (pts (xy 152.4 125.73) (xy 152.4 153.67))
+  (wire (pts (xy 152.4 125.73) (xy 152.4 138.43))
     (stroke (width 0) (type default) (color 0 0 0 0))
   )
@@
     (stroke (width 0) (type default) (color 0 0 0 0))
   )
+  (wire (pts (xy 135.89 110.49) (xy 151.13 110.49))
+    (stroke (width 0) (type default) (color 0 0 0 0))
+  )
   (wire (pts (xy 135.89 156.21) (xy 144.78 156.21))
     (stroke (width 0) (type default) (color 0 0 0 0))
@@
     (stroke (width 0) (type default) (color 0 0 0 0))
   )
+  (wire (pts (xy 135.89 138.43) (xy 152.4 138.43))
+    (stroke (width 0) (type default) (color 0 0 0 0))
+  )
   (wire (pts (xy 219.71 35.56) (xy 210.82 35.56))
     (stroke (width 0) (type default) (color 0 0 0 0))
@@
     (stroke (width 0) (type default) (color 0 0 0 0))
   )
+  (wire (pts (xy 83.82 151.13) (xy 83.82 163.83))
+    (stroke (width 0) (type default) (color 0 0 0 0))
+  )
   (wire (pts (xy 176.53 149.86) (xy 185.42 149.86))
     (stroke (width 0) (type default) (color 0 0 0 0))
@@
     (stroke (width 0) (type default) (color 0 0 0 0))
   )
+  (wire (pts (xy 152.4 153.67) (xy 152.4 163.83))
+    (stroke (width 0) (type default) (color 0 0 0 0))
+  )
   (wire (pts (xy 100.33 120.65) (xy 91.44 120.65))
     (stroke (width 0) (type default) (color 0 0 0 0))
@@
     (stroke (width 0) (type default) (color 0 0 0 0))
   )
+  (wire (pts (xy 151.13 110.49) (xy 151.13 91.44))
+    (stroke (width 0) (type default) (color 0 0 0 0))
+  )
   (wire (pts (xy 100.33 153.67) (xy 91.44 153.67))
     (stroke (width 0) (type default) (color 0 0 0 0))
@@
     (stroke (width 0) (type default) (color 0 0 0 0))
   )
-  (wire (pts (xy 149.86 88.9) (xy 157.48 88.9))
-    (stroke (width 0) (type default) (color 0 0 0 0))
-  )
   (wire (pts (xy 100.33 115.57) (xy 91.44 115.57))
     (stroke (width 0) (type default) (color 0 0 0 0))
   )
+  (wire (pts (xy 100.33 125.73) (xy 83.82 125.73))
+    (stroke (width 0) (type default) (color 0 0 0 0))
+  )
   (wire (pts (xy 100.33 156.21) (xy 91.44 156.21))
     (stroke (width 0) (type default) (color 0 0 0 0))
@@
     (stroke (width 0) (type default) (color 0 0 0 0))
   )
-  (wire (pts (xy 147.32 110.49) (xy 149.86 110.49))
-    (stroke (width 0) (type default) (color 0 0 0 0))
-  )
   (wire (pts (xy 135.89 130.81) (xy 144.78 130.81))
     (stroke (width 0) (type default) (color 0 0 0 0))
@@
     (stroke (width 0) (type default) (color 0 0 0 0))
   )
+  (wire (pts (xy 83.82 113.03) (xy 83.82 125.73))
+    (stroke (width 0) (type default) (color 0 0 0 0))
+  )
   (wire (pts (xy 200.66 111.76) (xy 198.12 111.76))
     (stroke (width 0) (type default) (color 0 0 0 0))
@@
     (stroke (width 0) (type default) (color 0 0 0 0))
   )
+  (wire (pts (xy 100.33 113.03) (xy 83.82 113.03))
+    (stroke (width 0) (type default) (color 0 0 0 0))
+  )
   (wire (pts (xy 100.33 123.19) (xy 91.44 123.19))
     (stroke (width 0) (type default) (color 0 0 0 0))
   )
+  (wire (pts (xy 83.82 125.73) (xy 83.82 138.43))
+    (stroke (width 0) (type default) (color 0 0 0 0))
+  )
+  (wire (pts (xy 83.82 163.83) (xy 152.4 163.83))
+    (stroke (width 0) (type default) (color 0 0 0 0))
+  )
   (wire (pts (xy 176.53 48.26) (xy 185.42 48.26))
     (stroke (width 0) (type default) (color 0 0 0 0))
@@
   )
   (wire (pts (xy 135.89 135.89) (xy 144.78 135.89))
+    (stroke (width 0) (type default) (color 0 0 0 0))
+  )
+  (wire (pts (xy 100.33 151.13) (xy 83.82 151.13))
+    (stroke (width 0) (type default) (color 0 0 0 0))
+  )
+  (wire (pts (xy 135.89 151.13) (xy 152.4 151.13))
     (stroke (width 0) (type default) (color 0 0 0 0))
   )
@@
     (pin "4")
   )
-  (symbol (lib_id "Diode:1N5817") (at 143.51 110.49 0) (unit 1)
-    (in_bom yes) (on_board yes) (fields_autoplaced)
-    (property "Reference" "D1" (id 0) (at 143.1925 104.14 0))
-    (property "Value" "1N5817" (id 1) (at 143.1925 106.68 0))
-    (property "Footprint" "Diode_THT:D_DO-41_SOD81_P10.16mm_Horizontal" (id 2) (at 143.51 114.935 0)
-      (effects (font (size 1.27 1.27)) hide)
-    )
-    (property "Datasheet" "http://www.vishay.com/docs/88525/1n5817.pdf" (id 3) (at 143.51 110.49 0)
-      (effects (font (size 1.27 1.27)) hide)
-    )
-    (pin "1")
-    (pin "2")
-  )
   (sheet_instances
     (path "/" (page "1"))
@@
       (reference "#PWR01") (unit 1) (value "GND") (footprint "")
     )
-    (path "/f372f267-8816-4f57-9137-fd0a8ff55b57"
-      (reference "D1") (unit 1) (value "1N5817") (footprint "Diode_THT:D_DO-41_SOD81_P10.16mm_Horizontal")
-    )
     (path "/f340092b-05f1-4654-bdfd-97debce52df0"
